File: recruitment.kicad_pcb (KiCad board)
At the start: 2 copper layers, 1 part

Commit message: set title block and JLCPCB design rules
Parts:
- removed C1: 1F, Capacitor_SMD:C_0805_2012Metric
Routing:
- net Net-(C1-Pad1): track 57.5 -> 0.00 mm
