File: recruitment.kicad_pcb (KiCad board)
At the start: 2 copper layers, 100 x 70 mm, 57 parts, among them J201 Micro-Fit 2P, J301 LOAD_IN, J302 LOAD_OUT, K301 G9EJ-1-P-E-UVD DC12, Q201 Si2319CDS, Q301 BCP56-16, Q302 BC847B, SW401 TEST, U201 TPS7B6933-Q1, U401 ACS781LLRTR-050B-T, U501 TLV1702, U502 MAX809S, U503 74LVC00

Commit message: Clean up silkscreen and add board markings
Other:
- board text added: "+3V3"
- board text added: "+VIN_PROT"
- board text added: "9-17V"
- board text added: "COIL_RS"
- board text added: "E-Agle TRT - Overcurrent monitor 500W"
- board text added: "FAULT_N"
- board text added: "GND"
- board text added: "LOAD IN 24-48V"
- board text added: "LOAD OUT"
- board text added: "PWR"
- board text added: "RELAY"
- board text added: "TEST"
- board text added: "TRIP"
- board text added: "V_SENSE"
- board text added: "Vth_Hi"
