File: power.kicad_sch (KiCad schematic)
At the start: 0 parts

Commit message: Add power supply sheet
Parts:
- added C201: 10µF 50V, Capacitor_SMD:C_1210_3225Metric, symbol Device:C
- added C202: 100nF 50V, Capacitor_SMD:C_0603_1608Metric, symbol Device:C
- added C203: 1µF 50V, Capacitor_SMD:C_0805_2012Metric, symbol Device:C
- added C204: 10µF 16V, Capacitor_SMD:C_0805_2012Metric, symbol Device:C
- added C205: 100nF 16V, Capacitor_SMD:C_0603_1608Metric, symbol Device:C
- added D201: SMBJ18CA, Diode_SMD:D_SMB, symbol Device:D_TVS
- added D202: 12V, Diode_SMD:D_SOD-123, symbol Device:D_Zener
- added D203: PWR yellow-green, LED_SMD:LED_0603_1608Metric, symbol Device:LED
- added F201: 0.5A 30V, Fuse:Fuse_1812_4532Metric, symbol Device:Polyfuse
- added J201: Micro-Fit 2P, Connector_Molex:Molex_Micro-Fit_3.0_43650-0215_1x02_P3.00mm_Vertical, symbol Connector_Generic:Conn_01x02
- added Q201: Si2319CDS, Package_TO_SOT_SMD:SOT-23, symbol Transistor_FET:Si2319CDS
- added R201: 100k, Resistor_SMD:R_0603_1608Metric, symbol Device:R
- added R202: 1k, Resistor_SMD:R_0603_1608Metric, symbol Device:R
- added TP201: +VIN_PROT, TestPoint:TestPoint_Pad_D1.5mm, symbol Connector:TestPoint
- added TP202: +3V3, TestPoint:TestPoint_Pad_D1.5mm, symbol Connector:TestPoint
- added TP203: GND, TestPoint:TestPoint_Keystone_5000-5004_Miniature, symbol Connector:TestPoint
- added U201: TPS7B6933-Q1, Package_TO_SOT_SMD:SOT-223-3_TabPin2, symbol monitor:TPS7B6933-Q1
Connections:
- new net: D203.2 (A), R202.2
- new net +3V3: C204.1, C205.1, R202.1, TP202.1, U201.3 (VO)
- new net +VIN_PROT: C201.1, C202.1, C203.1, D202.1 (K), Q201.2 (S), TP201.1, U201.1 (VI)
- new net GND: C201.2, C202.2, C203.2, C204.2, C205.2, D201.2 (A2), D203.1 (K), J201.2 (Pin_2), R201.2, TP203.1, U201.2 (GND)
- new net Q201_G: D202.2 (A), Q201.1 (G), R201.1
- new net VIN_FUSED: D201.1 (A1), F201.2, Q201.3 (D)
- new net VIN_RAW: F201.1, J201.1 (Pin_1)
